File: induction_encoder.kicad_pcb (KiCad board)
At the start: 4 copper layers, 170 x 170 mm, 62 parts, among them J2 Conn_01x06, U1 MT9105ET, U10 IPS2200, U11 ADS1115IDGS, U12 ADS1115IDGS, U2 MT9105ET, U3 MT9105ET, U4 MT9105ET, U5 MT9105ET, U6 MT9105ET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

Commit message: starting layout for 118-220mm induction encoder
Parts:
- moved JP1 231.1 mm to (344.8, 278.0), turned to 180 degrees
- moved TP1 218.9 mm to (361.7, 260.0)
- moved J2 218.3 mm to (347.8, 284.0)
- moved C12 215.9 mm to (329.1, 305.9)
- moved C8 215.9 mm to (332.6, 302.5)
- moved U2 215.9 mm to (330.5, 303.9)
- moved TP4 214.8 mm to (353.5, 256.9)
- moved JP2 212.9 mm to (354.1, 236.7)
- moved TP8 212.7 mm to (353.9, 234.7)
- moved C26 209.8 mm to (358.8, 234.2)
- moved C27 209.8 mm to (358.8, 239.1)
- moved U9 209.8 mm to (358.4, 236.7)
- moved C16 208.0 mm to (260.9, 332.2)
- moved C9 208.0 mm to (265.8, 332.2)
- moved U4 208.0 mm to (263.4, 331.7)
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Routing:
- net (no net): track 1900.4 -> 0.00 mm, vias 10 -> 0
- net TX+: track 11.8 -> 1730.2 mm, vias 1 -> 2
- net 1+: track 8.37 -> 1110.0 mm, vias 0 -> 8
- net 2: track 746.1 -> 1044.2 mm
- net /MAG5: track 190.5 -> 7.87 mm
- net /MAG6: track 148.4 -> 14.0 mm
- net /MAG4: track 111.5 -> 1.77 mm
- net 1-: track 9.10 -> 82.9 mm
- net /MAG1: track 78.2 -> 10.2 mm
- net /MAG7: track 71.8 -> 9.08 mm
- net /MAG3: track 58.2 -> 3.18 mm
- net TX-: track 8.13 -> 38.8 mm
- net +3V3: track 20.6 -> 19.6 mm
- net /MAG2: vias 1 -> 0
- removed copper zone on In2.Cu, net GND
Other:
- board size 170 x 170 mm -> 220 x 220 mm
- board text added: "Induction Encoder Int D: 118mm Out D: 220mm December 2024"

Commit message: 118-220 layout progress
Parts:
- moved TP1 16.6 mm to (363.9, 243.5)
- moved TP8 11.5 mm to (358.5, 224.2)
- moved C1 7.63 mm to (336.6, 175.6), turned to 90 degrees
- moved C4 7.39 mm to (335.1, 175.6), turned to -90 degrees
- moved TP7 0.61 mm to (349.8, 205.3)
Routing:
- net /MAG5: track 7.87 -> 316.0 mm
- net /MAG6: track 14.0 -> 243.4 mm
- net /MAG4: track 1.77 -> 164.6 mm
- net /MAG7: track 9.08 -> 144.5 mm, vias 1 -> 0
- net SDA: track 35.8 -> 136.7 mm, vias 2 -> 5
- net SCL: track 32.8 -> 130.2 mm, vias 2 -> 5
- net /MAG3: track 3.18 -> 87.0 mm
- net /MAG1: track 10.2 -> 83.2 mm, vias 1 -> 0
- net /MAG8: track 8.29 -> 68.4 mm
- net +3V3: track 19.6 -> 36.7 mm, vias 0 -> 4
- net /MAG2: track 2.81 -> 12.8 mm
- net GND: track 76.6 -> 78.4 mm, vias 36 -> 37
- net TX+: track 1730.2 -> 1731.3 mm, vias 2 -> 3
- net 2: track 1044.2 -> 1045.3 mm
- net 1-: track 82.9 -> 83.8 mm
- added copper zone on In2.Cu, net GND

Commit message: 118-220 boards ready to order
Parts:
- R10: value 10k -> 10K
- moved JP2 0.66 mm to (354.4, 237.3), turned to -90 degrees
- moved JP1 0.34 mm to (345.1, 278.2)
Routing:
- net RDY: track 1.57 -> 96.9 mm
- net +3V3: track 36.7 -> 39.5 mm
- net TX+: track 1731.3 -> 1732.1 mm
Other:
- outline, holes or cut-outs redrawn
- board text added: "1+"
- board text added: "3V3"
- board text added: "RDY"
- board text added: "SCL"
- board text added: "SDA"
- board text added: "TX+"
